File: leftSideGenerated/keyboard-layout.kicad_pcb (KiCad board)
At the start: 2 copper layers, 136.4 x 101.2 mm, 56 parts

Commit message: shit ton of files
Parts:
- added REF**: NRF51822, ZelaFoots:NRF51822, F.Cu at (0.76, 72.6)
Changed lines of the file:
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@@
     (tracks 213)
     (zones 0)
-    (modules 56)
+    (modules 57)
     (nets 122)
   )
@@
     (42 Eco1.User user)
     (43 Eco2.User user)
-    (44 Edge.Cuts user)
+    (44 Edge.Cuts user hide)
     (45 Margin user)
     (46 B.CrtYd user hide)
@@
     (add_net "Net-(K_Z-Pad4)")
   )
+  (module ZelaFoots:NRF51822 (layer F.Cu)
+    (at 0.762 72.644)
+    (fp_text reference REF** (at 1.016 8.128) (layer F.SilkS)
+      (effects (font (size 1 1) (thickness 0.15)))
+    )
+    (fp_text value NRF51822 (at 0.3 -16.1) (layer F.Fab)
+      (effects (font (size 1 1) (thickness 0.15)))
+    )
+    (fp_poly (pts (xy -13 -12.9) (xy 12 -12.9) (xy 12 5) (xy -13 5)) (layer B.SilkS) (width 0.1))
+    (fp_line (start 12 5) (end 12 -12.9) (layer F.SilkS) (width 0.12))
+    (fp_line (start 12 -12.9) (end -13 -12.9) (layer F.SilkS) (width 0.12))
+    (fp_line (start -13 -12.9) (end -13 5) (layer F.SilkS) (width 0.12))
+    (fp_line (start -13 5) (end 12 5) (layer F.SilkS) (width 0.12))
+    (pad 1 thru_hole circle (at -11.7 -12) (size 1.524 1.524) (drill 0.762) (layers *.Cu *.Mask))
+    (pad 2 thru_hole circle (at -9.7 -12) (size 1.524 1.524) (drill 0.762) (layers *.Cu *.Mask))
+    (pad 3 thru_hole circle (at -11.7 -10) (size 1.524 1.524) (drill 0.762) (layers *.Cu *.Mask))
+    (pad 4 thru_hole circle (at -9.7 -10) (size 1.524 1.524) (drill 0.762) (layers *.Cu *.Mask))
+    (pad 5 thru_hole circle (at -11.7 -8) (size 1.524 1.524) (drill 0.762) (layers *.Cu *.Mask))
+    (pad 6 thru_hole circle (at -9.7 -8) (size 1.524 1.524) (drill 0.762) (layers *.Cu *.Mask))
+    (pad 7 thru_hole circle (at -11.7 -6) (size 1.524 1.524) (drill 0.762) (layers *.Cu *.Mask))
+    (pad 8 thru_hole circle (at -9.7 -6) (size 1.524 1.524) (drill 0.762) (layers *.Cu *.Mask))
+    (pad 9 thru_hole circle (at -11.7 -4) (size 1.524 1.524) (drill 0.762) (layers *.Cu *.Mask))
+    (pad 10 thru_hole circle (at -9.7 -4) (size 1.524 1.524) (drill 0.762) (layers *.Cu *.Mask))
+    (pad 11 thru_hole circle (at -11.7 -2) (size 1.524 1.524) (drill 0.762) (layers *.Cu *.Mask))
+    (pad 12 thru_hole circle (at -9.7 -2) (size 1.524 1.524) (drill 0.762) (layers *.Cu *.Mask))
+    (pad 13 thru_hole circle (at -11.7 0) (size 1.524 1.524) (drill 0.762) (layers *.Cu *.Mask))
+    (pad 14 thru_hole circle (at -9.7 0) (size 1.524 1.524) (drill 0.762) (layers *.Cu *.Mask))
+    (pad 15 thru_hole circle (at -11.7 2) (size 1.524 1.524) (drill 0.762) (layers *.Cu *.Mask))
+    (pad 16 thru_hole circle (at -9.7 2) (size 1.524 1.524) (drill 0.762) (layers *.Cu *.Mask))
+    (pad 17 thru_hole circle (at -11.6 4) (size 1.524 1.524) (drill 0.762) (layers *.Cu *.Mask))
+    (pad 18 thru_hole circle (at -9.6 4) (size 1.524 1.524) (drill 0.762) (layers *.Cu *.Mask))
+    (pad 20 thru_hole circle (at 8.3 -12) (size 1.524 1.524) (drill 0.762) (layers *.Cu *.Mask))
+    (pad 19 thru_hole circle (at 10.3 -12) (size 1.524 1.524) (drill 0.762) (layers *.Cu *.Mask))
+    (pad 21 thru_hole circle (at 8.3 -10) (size 1.524 1.524) (drill 0.762) (layers *.Cu *.Mask))
+    (pad 22 thru_hole circle (at 10.3 -10) (size 1.524 1.524) (drill 0.762) (layers *.Cu *.Mask))
+    (pad 23 thru_hole circle (at 8.3 -8) (size 1.524 1.524) (drill 0.762) (layers *.Cu *.Mask))
+    (pad 24 thru_hole circle (at 10.3 -8) (size 1.524 1.524) (drill 0.762) (layers *.Cu *.Mask))
+    (pad 25 thru_hole circle (at 8.3 -6) (size 1.524 1.524) (drill 0.762) (layers *.Cu *.Mask))
+    (pad 26 thru_hole circle (at 10.3 -6) (size 1.524 1.524) (drill 0.762) (layers *.Cu *.Mask))
+    (pad 27 thru_hole circle (at 8.3 -4) (size 1.524 1.524) (drill 0.762) (layers *.Cu *.Mask))
+    (pad 28 thru_hole circle (at 10.3 -4) (size 1.524 1.524) (drill 0.762) (layers *.Cu *.Mask))
+    (pad 29 thru_hole circle (at 8.3 -2) (size 1.524 1.524) (drill 0.762) (layers *.Cu *.Mask))
+    (pad 30 thru_hole circle (at 10.3 -2) (size 1.524 1.524) (drill 0.762) (layers *.Cu *.Mask))
+    (pad 31 thru_hole circle (at 8.3 0) (size 1.524 1.524) (drill 0.762) (layers *.Cu *.Mask))
+    (pad 32 thru_hole circle (at 10.3 0) (size 1.524 1.524) (drill 0.762) (layers *.Cu *.Mask))
+    (pad 33 thru_hole circle (at 8.3 2) (size 1.524 1.524) (drill 0.762) (layers *.Cu *.Mask))
+    (pad 34 thru_hole circle (at 10.2 2) (size 1.524 1.524) (drill 0.762) (layers *.Cu *.Mask))
+    (pad 35 thru_hole circle (at 8.3 4) (size 1.524 1.524) (drill 0.762) (layers *.Cu *.Mask))
+    (pad 36 thru_hole circle (at 10.3 4) (size 1.524 1.524) (drill 0.762) (layers *.Cu *.Mask))
+  )
   (module MX_Alps_Hybrid:MX-1U-NoLED (layer F.Cu)
