File: leftSideGenerated/keyboard-layout.sch (KiCad schematic (older format))
At the start: 56 parts

Commit message: shit ton of files
Parts:
- removed K_, K_1, K_2, K_3, K_4, K_5, K_6, K_A, K_ALT, K_C, K_CAPS_LOCK, K_CTRL, K_D, K_E, K_ESC, K_F, K_G, K_MOD, K_Q, K_R, K_S, K_SHIFT, K_T, K_TAB, K_V, K_W, K_X, K_Z: D, keyboard_parts:D_SOD123_axial, symbol Device:D
- removed K_: KEYSW, MX_Alps_Hybrid:MX-2.75U-NoLED, symbol keyboard_parts:KEYSW
- removed K_A, K_C, K_D, K_E, K_ESC, K_F, K_G, K_Q, K_R, K_S, K_T, K_V, K_W, K_X, K_Z: KEYSW, MX_Alps_Hybrid:MX-1U-NoLED, symbol keyboard_parts:KEYSW
- removed K_ALT, K_CTRL, K_MOD: KEYSW, MX_Alps_Hybrid:MX-1.25U-NoLED, symbol keyboard_parts:KEYSW
- removed K_CAPS_LOCK: KEYSW, MX_Alps_Hybrid:MX-1.75U-NoLED, symbol keyboard_parts:KEYSW
- removed K_SHIFT: KEYSW, MX_Alps_Hybrid:MX-2.25U-NoLED, symbol keyboard_parts:KEYSW
- removed K_TAB: KEYSW, MX_Alps_Hybrid:MX-1.5U-NoLED, symbol keyboard_parts:KEYSW
- added D_1, D_2, D_3, D_4, D_5, D_6, D_7, D_A1, D_ALT1, D_C1, D_CAPS_LOCK1, D_CTRL1, D_D1, D_E1, D_ESC1, D_F1, D_G1, D_MOD1, D_Q1, D_R1, D_S1, D_SHIFT1, D_T1, D_TAB1, D_V1, D_W1, D_X1, D_Z1: D, keyboard_parts:D_SOD123_axial, symbol Device:D
- added K_7: KEYSW, MX_Alps_Hybrid:MX-2.75U-NoLED, symbol keyboard_parts:KEYSW
- added K_A1, K_C1, K_D1, K_E1, K_ESC1, K_F1, K_G1, K_Q1, K_R1, K_S1, K_T1, K_V1, K_W1, K_X1, K_Z1: KEYSW, MX_Alps_Hybrid:MX-1U-NoLED, symbol keyboard_parts:KEYSW
- added K_ALT1, K_CTRL1, K_MOD1: KEYSW, MX_Alps_Hybrid:MX-1.25U-NoLED, symbol keyboard_parts:KEYSW
- added K_CAPS_LOCK1: KEYSW, MX_Alps_Hybrid:MX-1.75U-NoLED, symbol keyboard_parts:KEYSW
- added K_SHIFT1: KEYSW, MX_Alps_Hybrid:MX-2.25U-NoLED, symbol keyboard_parts:KEYSW
- added K_TAB1: KEYSW, MX_Alps_Hybrid:MX-1.5U-NoLED, symbol keyboard_parts:KEYSW
- added U1: NRF51822, ZelaFoots:NRF51822, symbol custom:NRF51822
Connections:
- net col0: now also K_CAPS_LOCK1.1, K_CTRL1.1, K_ESC1.1, K_SHIFT1.1, K_TAB1.1, U1.~ (VCC)
- net col1: now also K_A1.1, K_MOD1.1, K_Q1.1, K_Z1.1, U1.~ (VCC)
- net col2: now also K_ALT1.1, K_S1.1, K_W1.1, K_X1.1, U1.~ (VCC)
- net col3: now also K_7.1, K_C1.1, K_D1.1, K_E1.1, U1.~ (VCC)
- net col4: now also K_F1.1, K_R1.1, K_V1.1, U1.~ (VCC)
- net col5: now also K_G1.1, K_T1.1, U1.~ (VCC)
- net col6: now also U1.~ (VCC)
- net row0: now also D_1.1 (K), D_2.1 (K), D_3.1 (K), D_4.1 (K), D_5.1 (K), D_6.1 (K), D_ESC1.1 (K), U1.~ (VCC)
- net row1: now also D_E1.1 (K), D_Q1.1 (K), D_R1.1 (K), D_T1.1 (K), D_TAB1.1 (K), D_W1.1 (K), U1.~ (VCC)
- net row2: now also D_A1.1 (K), D_CAPS_LOCK1.1 (K), D_D1.1 (K), D_F1.1 (K), D_G1.1 (K), D_S1.1 (K)
- net row3: now also D_C1.1 (K), D_SHIFT1.1 (K), D_V1.1 (K), D_X1.1 (K), D_Z1.1 (K), U1.~ (VCC)
- net row4: now also D_7.1 (K), D_ALT1.1 (K), D_CTRL1.1 (K), D_MOD1.1 (K), U1.~ (VCC)
- net at K_1.2: now also D_1.2 (A)
- net at K_2.2: now also D_2.2 (A)
- net at K_3.2: now also D_3.2 (A)
- net at K_4.2: now also D_4.2 (A)
- net at K_5.2: now also D_5.2 (A)
- net at K_6.2: now also D_6.2 (A)
- new net: D_A1.2 (A), K_A1.2
- new net: D_Z1.2 (A), K_Z1.2
- new net: D_SHIFT1.2 (A), K_SHIFT1.2
- new net: D_F1.2 (A), K_F1.2
- new net: D_E1.2 (A), K_E1.2
- new net: D_ALT1.2 (A), K_ALT1.2
- new net: D_CTRL1.2 (A), K_CTRL1.2
- new net: D_V1.2 (A), K_V1.2
- new net: D_S1.2 (A), K_S1.2
- new net: D_MOD1.2 (A), K_MOD1.2
- new net: D_7.2 (A), K_7.2
- new net: D_G1.2 (A), K_G1.2
- new net: D_ESC1.2 (A), K_ESC1.2
- new net: D_Q1.2 (A), K_Q1.2
- new net: D_C1.2 (A), K_C1.2
- new net: D_T1.2 (A), K_T1.2
- new net: D_W1.2 (A), K_W1.2
- new net: D_CAPS_LOCK1.2 (A), K_CAPS_LOCK1.2
- new net: D_X1.2 (A), K_X1.2
- new net: D_D1.2 (A), K_D1.2
- new net: D_R1.2 (A), K_R1.2
- new net: D_TAB1.2 (A), K_TAB1.2
- no-connect marks 0 -> 25
