File: FINALPCB/CASE_LASER_FINAL.kicad_pcb (KiCad board)
At the start: 2 copper layers, 295.1 x 256.2 mm, 0 parts

Commit message: rip and done
Other:
- board size 295.1 x 256.2 mm -> 134.1 x 189.7 mm
